Commit message: proper kinematics for BarrettHand BH-280

File: barrett_hand_defs/defs/barret_hand.urdf.xacro (robot description, xacro)
@@ -52,12 +52,4 @@
             </geometry>
           </collision>
-<!--
-          <self_collision_checking>
-            <origin xyz="0 0 0.04" rpy="0 0 0"/>
-            <geometry>
-              <capsule radius="0.05" length="0.04"/>
-            </geometry>
-          </self_collision_checking>
--->
           <self_collision_checking>
             <origin xyz="0 0 0" rpy="0 0 0"/>
@@ -73,9 +65,4 @@
                 <point xyz="0.06 0 0" frame="${prefix}_HandFingerTwoKnuckleOneLink"/>
                 <point xyz="0 -0.06 0.06" frame="${prefix}_HandPalmLink"/>
-                <!-- proximal fingers' links -->
-<!--                <point xyz="0 0 0" frame="${prefix}_HandFingerOneKnuckleTwoLink"/>
-                <point xyz="0 0 0" frame="${prefix}_HandFingerTwoKnuckleTwoLink"/>
-                <point xyz="0 0 0" frame="${prefix}_HandFingerThreeKnuckleTwoLink"/>
--->
                 <!-- distal fingers' links -->
                 <point xyz="0 0 0" frame="${prefix}_HandFingerOneKnuckleThreeLink"/>
@@ -172,5 +159,5 @@
             <axis xyz="0 0 -1"/>
                             <!-- 122 degrees - start orientation of 0.4 degrees-->
-            <limit effort="1" lower="0" upper="${2.12930169 - 0.00698131701}" velocity="3.27"/>
+            <limit effort="1" lower="0" upper="2.443388889" velocity="3.27"/>
             <dynamics damping="0.005" friction="100.0"/>
         </joint>
@@ -208,9 +195,9 @@
             <parent link="${prefix}_HandFinger${number}KnuckleTwoLink"/>
             <child link="${prefix}_HandFinger${number}KnuckleThreeLink"/>
-                                        <!-- 42 degrees -->
-            <origin xyz="0.07 0 0" rpy="0 0 -0.733038286"/>
+                                        <!-- 39.56 degrees -->
+            <origin xyz="0.07 0 0" rpy="0 0 -0.690452252"/>
             <axis xyz="0 0 -1"/>
                                 <!-- measured max angle is 94.  so upper limit is 94 - start orientation (42 degrees)-->
-            <limit effort="1" lower="0" upper="${1.6406095 - 0.733038286}" velocity="3.27"/>
+            <limit effort="1" lower="0" upper="0.837733333" velocity="3.27"/>
             <dynamics damping="0.005" friction="100.0"/>
         </joint>
@@ -224,9 +211,10 @@
             <insert_block name="origin"/>
         </xacro:palm>
-        <xacro:fingers prefix="${prefix}" parent="${prefix}_HandPalmLink" number="Three" xyz="0 -0.05 0.0801966" rpy="-${0.5 * PI} -0.0429350996 -${0.5 * PI}"/>
+        <xacro:fingers prefix="${prefix}" parent="${prefix}_HandPalmLink" number="Three" xyz="0 -0.05 0.0754" rpy="-${0.5 * PI} 0 -${0.5 * PI}"/>
         <xacro:KnuckleOne prefix="${prefix}" number="One" xyz=".02497 0 0.0587966" rpy="0 0 ${0.5 * PI}" axis="0 0 -1"/>
-        <xacro:fingers prefix="${prefix}" parent="${prefix}_HandFingerOneKnuckleOneLink" number="One" xyz=".05 0 0.02140" rpy="-${0.5 * PI} -0.0429350996 0"/>
+        <xacro:fingers prefix="${prefix}" parent="${prefix}_HandFingerOneKnuckleOneLink" number="One" xyz=".05 0 0.0166034" rpy="-${0.5 * PI} 0 0"/>
         <xacro:KnuckleOne prefix="${prefix}" number="Two" xyz="-.02497 0 0.0587966" rpy="0 0 ${0.5 * PI}" axis ="0 0 1"/>
-        <xacro:fingers prefix="${prefix}" parent="${prefix}_HandFingerTwoKnuckleOneLink" number="Two" xyz=".05 0 0.02140" rpy="-${0.5 * PI} -0.0429350996 0"/>
+        <xacro:fingers prefix="${prefix}" parent="${prefix}_HandFingerTwoKnuckleOneLink" number="Two" xyz=".05 0 0.0166034" rpy="-${0.5 * PI} 0 0"/>
+<!--        <xacro:fingers prefix="${prefix}" parent="${prefix}_HandFingerTwoKnuckleOneLink" number="Two" xyz=".05 0 0.0166034" rpy="-${0.5 * PI} -0.0429350996 0"/>-->
 </xacro:macro>
 </robot>

Commit message: options for collision model

File: barrett_hand_defs/defs/barret_hand.urdf.xacro (robot description, xacro)
@@ -28,183 +28,238 @@
        xmlns:interface="http://playerstage.sourceforge.net/gazebo/xmlschema/#interface"
        xmlns:xacro="http://www.ros.org/wiki/xacro">
-    <xacro:property name="homeDirectory" value="package://barrett_hand_defs" />
-    <xacro:property name="highResModelDirectory" value="${homeDirectory}/meshes/splitModels" />
-    <xacro:property name="PI" value="3.1415926535897931" />
-    <xacro:macro name="palm" params="prefix parent *origin">
-        <link name="${prefix}_HandPalmLink" >
-          <inertial>
-            <origin xyz="0.00035500 -0.00499005 0.04864979" />
-            <mass value="0.63352875" />
-            <inertia  ixx="0.00102103" ixy="0.00000775"  ixz="-0.00001230"
-                                       iyy="0.00080944"  iyz="-0.00014417"
-                                                         izz="0.00068788" />
-          </inertial>
-          <visual>
-            <origin xyz="0 0 0" rpy="${PI} 0 0" />
-            <geometry>
-                    <mesh filename="${homeDirectory}/meshes/HandPalmLink.dae"/>
-            </geometry>
-          </visual>
-          <collision>
-            <origin xyz="0 0 0" rpy="0 0 0" />
-            <geometry>
-              <mesh filename="${homeDirectory}/meshes/palm.stl"/>
-            </geometry>
-          </collision>
-          <self_collision_checking>
-            <origin xyz="0 0 0" rpy="0 0 0"/>
-            <geometry>
-              <convex>
-                <!-- gripper base points -->
-                <point xyz="0.03 0.03 0.0" frame="${prefix}_HandPalmLink"/>
-                <point xyz="-0.03 0.03 0.0" frame="${prefix}_HandPalmLink"/>
-                <point xyz="-0.03 -0.03 0.0" frame="${prefix}_HandPalmLink"/>
-                <point xyz="0.03 -0.03 0.0" frame="${prefix}_HandPalmLink"/>
-                <!-- fingers' base links -->
-                <point xyz="0.06 0 0" frame="${prefix}_HandFingerOneKnuckleOneLink"/>
-                <point xyz="0.06 0 0" frame="${prefix}_HandFingerTwoKnuckleOneLink"/>
-                <point xyz="0 -0.06 0.06" frame="${prefix}_HandPalmLink"/>
-                <!-- distal fingers' links -->
-                <point xyz="0 0 0" frame="${prefix}_HandFingerOneKnuckleThreeLink"/>
-                <point xyz="0 0 0" frame="${prefix}_HandFingerTwoKnuckleThreeLink"/>
-                <point xyz="0 0 0" frame="${prefix}_HandFingerThreeKnuckleThreeLink"/>
-                <point xyz="0.06 0 0" frame="${prefix}_HandFingerOneKnuckleThreeLink"/>
-                <point xyz="0.06 0 0" frame="${prefix}_HandFingerTwoKnuckleThreeLink"/>
-                <point xyz="0.06 0 0" frame="${prefix}_HandFingerThreeKnuckleThreeLink"/>
-              </convex>
-            </geometry>
-          </self_collision_checking>
-        </link>
-        <gazebo reference="${prefix}_HandPalmLink">
-          <turnGravityOff>true</turnGravityOff>
-        </gazebo>
-        <joint name="${prefix}_HandPalmJoint" type="fixed">
-            <parent link="${parent}"/>
-            <child link="${prefix}_HandPalmLink"/>
-            <insert_block name="origin"/>
-            <provideFeedback value="true"/>
-        </joint>
-    </xacro:macro>
-    <xacro:macro name="KnuckleOne" params="prefix number xyz rpy axis">
-        <link name="${prefix}_HandFinger${number}KnuckleOneLink">
-        <visual>
-            <origin xyz="0 0 -0.017" rpy="${0.5 * PI} 0 -${0.5 * PI}" />
-            <geometry>
-                <mesh filename="${homeDirectory}/meshes/KnuckleOneLink.dae"/>
-            </geometry>
-        </visual>
-        <inertial>
-            <origin xyz="0.03201666 -0.00086502 0.00890075" />
-            <mass value="0.16252678" />
-            <inertia  ixx="0.00002567" ixy="-0.00000146"  ixz="0.00001128"
-                    iyy="0.00008818"   iyz="-0.00000094"
-                    izz="0.00007827" />
-        </inertial>
-        <collision>
-            <origin xyz="0 0 0" rpy="${0.5 * PI} 0 -${0.5 * PI}" />
-            <geometry>
-                    <mesh filename="${homeDirectory}/meshes/firstFingerLink.stl"/>
-            </geometry>
-            <mu1 value="50000.0" />
-            <mu2 value="50000.0" />
-            <kp  value="1000000.0" />
-            <kd  value="1.0" />
-        </collision>
-        </link>
-        <gazebo reference="${prefix}_HandFinger${number}KnuckleOneLink">
-          <turnGravityOff>true</turnGravityOff>
-        </gazebo>
-        <joint name="${prefix}_HandFinger${number}KnuckleOneJoint" type="revolute">
-            <parent link="${prefix}_HandPalmLink"/>
-            <child link="${prefix}_HandFinger${number}KnuckleOneLink"/>
-            <origin xyz="${xyz}" rpy="${rpy}"/>
-            <axis xyz="${axis}"/>
-            <limit effort="1" lower="0" upper="${PI}" velocity="3.27"/>
-            <dynamics damping="0.05" friction="100.0"/>
-        </joint>
-    </xacro:macro>
- <xacro:macro name="KnuckleTwo" params="parent prefix number xyz rpy">
-        <link name="${prefix}_HandFinger${number}KnuckleTwoLink">
-            <visual>
-                <origin xyz="0 0 0" rpy="${PI} ${0.5 * PI} 0" />
-                <geometry>
-                    <mesh filename="${homeDirectory}/meshes/KnuckleTwoLink.dae"/>
-                </geometry>
-            </visual>
-            <inertial>
-                <origin xyz=".031720 .001070 -.000586" />
-                <mass value="0.057957" />
-                <inertia  ixx="0.00000461" ixy="0.00000003"  ixz="0.00000164"
-                                           iyy="0.00003590"  iyz="0.00000004"
-                                                             izz="0.00003682" />
-            </inertial>
-            <collision>
-                <origin xyz="0 0 0" rpy="${PI} ${0.5 * PI} 0" />
-                <geometry>
-                    <mesh filename="${homeDirectory}/meshes/secondFingerLink.stl"/>
-                </geometry>
-                <mu1 value="50000.0" />
-                <mu2 value="50000.0" />
-                <kp  value="1000000.0" />
-                <kd  value="1.0" />
-            </collision>
-        </link>
-        <gazebo reference="${prefix}_HandFinger${number}KnuckleTwoLink">
-          <turnGravityOff>true</turnGravityOff>
-        </gazebo>
-        <joint name="${prefix}_HandFinger${number}KnuckleTwoJoint" type="revolute">
-            <parent link="${parent}"/>
-            <child link="${prefix}_HandFinger${number}KnuckleTwoLink"/>
-            <origin xyz="${xyz}" rpy="${rpy}"/>
-            <axis xyz="0 0 -1"/>
-                            <!-- 122 degrees - start orientation of 0.4 degrees-->
-            <limit effort="1" lower="0" upper="2.443388889" velocity="3.27"/>
-            <dynamics damping="0.005" friction="100.0"/>
-        </joint>
-    </xacro:macro>
-    <xacro:macro name="KnuckleThree" params="prefix number">
-        <link name="${prefix}_HandFinger${number}KnuckleThreeLink">
-          <visual>
-            <origin xyz="0 0 0" rpy="0 ${0.5 * PI} 0" />
-            <geometry>
-                <mesh filename="${homeDirectory}/meshes/KnuckleThreeLink.dae"/>
-            </geometry>
-          </visual>
-          <inertial>
-            <origin xyz="0.01970974 0.00182016 0.00020041" />
-            <mass value="0.03421781" />
-            <inertia  ixx="0.00000287" ixy="0.00000091"  ixz="-0.00000007"
-                                       iyy="0.00001329"  iyz="-0.00000002"
-                                                         izz="0.00001214" />
-          </inertial>
-          <collision>
-            <origin xyz="0 0 0" rpy="0 ${0.5 * PI} 0" />
-            <geometry>
-                    <mesh filename="${homeDirectory}/meshes/thirdFingerLink.stl"/>
-            </geometry>
-            <mu1 value="50000.0" />
-            <mu2 value="50000.0" />
-            <kp  value="1000000.0" />
-            <kd  value="1.0" />
-          </collision>
-        </link>
-        <gazebo reference="${prefix}_HandFinger${number}KnuckleThreeLink">
-          <turnGravityOff>true</turnGravityOff>
-        </gazebo>
-        <joint name="${prefix}_HandFinger${number}KnuckleThreeJoint" type="revolute">
-            <parent link="${prefix}_HandFinger${number}KnuckleTwoLink"/>
-            <child link="${prefix}_HandFinger${number}KnuckleThreeLink"/>
-                                        <!-- 39.56 degrees -->
-            <origin xyz="0.07 0 0" rpy="0 0 -0.690452252"/>
-            <axis xyz="0 0 -1"/>
-                                <!-- measured max angle is 94.  so upper limit is 94 - start orientation (42 degrees)-->
-            <limit effort="1" lower="0" upper="0.837733333" velocity="3.27"/>
-            <dynamics damping="0.005" friction="100.0"/>
-        </joint>
-    </xacro:macro>
-    <xacro:macro name="fingers" params="parent prefix number xyz rpy">
-        <xacro:KnuckleTwo parent="${parent}" prefix="${prefix}" number="${number}" xyz="${xyz}" rpy="${rpy}" />
-        <xacro:KnuckleThree prefix="${prefix}" number="${number}"/>
-    </xacro:macro>
+  <xacro:arg name="collision_model_full" default="true"/>
+  <xacro:arg name="collision_model_simplified" default="false"/>
+  <xacro:arg name="collision_model_enlarged" default="false"/>
+  <xacro:property name="homeDirectory" value="package://barrett_hand_defs" />
+  <xacro:property name="highResModelDirectory" value="${homeDirectory}/meshes/splitModels" />
+  <xacro:property name="PI" value="3.1415926535897931" />
+  <property name="collision_model_enlargement" value="$(arg collision_model_enlargement)" />
+  <xacro:macro name="palm" params="prefix parent *origin">
+    <link name="${prefix}_HandPalmLink" >
+      <inertial>
+        <origin xyz="0.00035500 -0.00499005 0.04864979" />
+        <mass value="0.63352875" />
+        <inertia  ixx="0.00102103" ixy="0.00000775"  ixz="-0.00001230"
+                                   iyy="0.00080944"  iyz="-0.00014417"
+                                                     izz="0.00068788" />
+      </inertial>
+      <visual>
+        <origin xyz="0 0 0" rpy="${PI} 0 0" />
+        <geometry>
+          <mesh filename="${homeDirectory}/meshes/HandPalmLink.dae"/>
+        </geometry>
+      </visual>
+      <xacro:unless value="$(arg collision_model_no_hands)">
+      <!-- collision mesh used for whole arm motion planning -->
+      <xacro:if value="$(arg collision_model_simplified)">
+        <collision>
+          <origin xyz="0 0 0.045" rpy="0 0 0" />
+          <geometry>
+            <cylinder radius="${0.045+collision_model_enlargement}" length="0.09"/>
+          </geometry>
+        </collision>
+        <collision>
+          <origin xyz="0 -0.035 0.07" rpy="0 0 0" />
+          <geometry>
+            <box size="${0.025+collision_model_enlargement*2} ${0.08+collision_model_enlargement*2} ${0.05+collision_model_enlargement*2}"/>
+          </geometry>
+        </collision>
+      </xacro:if>
+      <!-- collision mesh used for grasp planning -->
+      <xacro:if value="$(arg collision_model_full)">
+        <collision>
+          <origin xyz="0 0 0" rpy="0 0 0" />
+          <geometry>
+            <mesh filename="${homeDirectory}/meshes/palm.stl"/>
+          </geometry>
+        </collision>
+      </xacro:if>
+      </xacro:unless>
+      <!-- collision mesh used for RT self-collision avoidance -->
+      <self_collision_checking>
+        <origin xyz="0 0 0" rpy="0 0 0"/>
+        <geometry>
+          <convex>
+            <!-- gripper base points -->
+            <point xyz="0.03 0.03 0.0" frame="${prefix}_HandPalmLink"/>
+            <point xyz="-0.03 0.03 0.0" frame="${prefix}_HandPalmLink"/>
+            <point xyz="-0.03 -0.03 0.0" frame="${prefix}_HandPalmLink"/>
+            <point xyz="0.03 -0.03 0.0" frame="${prefix}_HandPalmLink"/>
+            <!-- fingers' base links -->
+            <point xyz="0.06 0 0" frame="${prefix}_HandFingerOneKnuckleOneLink"/>
+            <point xyz="0.06 0 0" frame="${prefix}_HandFingerTwoKnuckleOneLink"/>
+            <point xyz="0 -0.06 0.06" frame="${prefix}_HandPalmLink"/>
+            <!-- distal fingers' links -->
+            <point xyz="0 0 0" frame="${prefix}_HandFingerOneKnuckleThreeLink"/>
+            <point xyz="0 0 0" frame="${prefix}_HandFingerTwoKnuckleThreeLink"/>
+            <point xyz="0 0 0" frame="${prefix}_HandFingerThreeKnuckleThreeLink"/>
+            <point xyz="0.06 0 0" frame="${prefix}_HandFingerOneKnuckleThreeLink"/>
+            <point xyz="0.06 0 0" frame="${prefix}_HandFingerTwoKnuckleThreeLink"/>
+            <point xyz="0.06 0 0" frame="${prefix}_HandFingerThreeKnuckleThreeLink"/>
+          </convex>
+        </geometry>
+      </self_collision_checking>
+    </link>
+    <gazebo reference="${prefix}_HandPalmLink">
+      <turnGravityOff>true</turnGravityOff>
+    </gazebo>
+    <joint name="${prefix}_HandPalmJoint" type="fixed">
+      <parent link="${parent}"/>
+      <child link="${prefix}_HandPalmLink"/>
+      <insert_block name="origin"/>
+      <provideFeedback value="true"/>
+    </joint>
+  </xacro:macro>
+  <xacro:macro name="KnuckleOne" params="prefix number xyz rpy axis">
+    <link name="${prefix}_HandFinger${number}KnuckleOneLink">
+      <visual>
+        <origin xyz="0 0 -0.017" rpy="${0.5 * PI} 0 -${0.5 * PI}" />
+        <geometry>
+          <mesh filename="${homeDirectory}/meshes/KnuckleOneLink.dae"/>
+        </geometry>
+      </visual>
+      <inertial>
+        <origin xyz="0.03201666 -0.00086502 0.00890075" />
+        <mass value="0.16252678" />
+        <inertia  ixx="0.00002567" ixy="-0.00000146"  ixz="0.00001128"
+                  iyy="0.00008818"   iyz="-0.00000094"
+                  izz="0.00007827" />
+      </inertial>
+      <xacro:unless value="$(arg collision_model_no_hands)">
+      <!-- collision mesh used for whole arm motion planning -->
+      <xacro:if value="$(arg collision_model_simplified)">
+        <collision>
+          <origin xyz="0.03 0 0.005" rpy="0 0 0" />
+          <geometry>
+            <box size="${0.08+collision_model_enlargement*2} ${0.025+collision_model_enlargement*2} ${0.05+collision_model_enlargement*2}"/>
+          </geometry>
+        </collision>
+      </xacro:if>
+      <!-- collision mesh used for grasp planning -->
+      <xacro:if value="$(arg collision_model_full)">
+        <collision>
+          <origin xyz="0 0 0" rpy="${0.5 * PI} 0 -${0.5 * PI}" />
+          <geometry>
+            <mesh filename="${homeDirectory}/meshes/firstFingerLink.stl"/>
+          </geometry>
+        </collision>
+      </xacro:if>
+      </xacro:unless>
+    </link>
+    <gazebo reference="${prefix}_HandFinger${number}KnuckleOneLink">
+      <turnGravityOff>true</turnGravityOff>
+    </gazebo>
+    <joint name="${prefix}_HandFinger${number}KnuckleOneJoint" type="revolute">
+      <parent link="${prefix}_HandPalmLink"/>
+      <child link="${prefix}_HandFinger${number}KnuckleOneLink"/>
+      <origin xyz="${xyz}" rpy="${rpy}"/>
+      <axis xyz="${axis}"/>
+      <limit effort="1" lower="0" upper="${PI}" velocity="3.27"/>
+      <dynamics damping="0.05" friction="100.0"/>
+    </joint>
+  </xacro:macro>
+  <xacro:macro name="KnuckleTwo" params="parent prefix number xyz rpy">
+    <link name="${prefix}_HandFinger${number}KnuckleTwoLink">
+      <visual>
+        <origin xyz="0 0 0" rpy="${PI} ${0.5 * PI} 0" />
+        <geometry>
+          <mesh filename="${homeDirectory}/meshes/KnuckleTwoLink.dae"/>
+        </geometry>
+      </visual>
+      <inertial>
+        <origin xyz=".031720 .001070 -.000586" />
+        <mass value="0.057957" />
+        <inertia  ixx="0.00000461" ixy="0.00000003"  ixz="0.00000164"
+                                   iyy="0.00003590"  iyz="0.00000004"
+                                                     izz="0.00003682" />
+      </inertial>
+      <xacro:unless value="$(arg collision_model_no_hands)">
+      <!-- collision mesh used for whole arm motion planning -->
+      <xacro:if value="$(arg collision_model_simplified)">
+        <collision>
+          <origin xyz="0.03 0 0" rpy="0 0 0" />
+          <geometry>
+            <box size="${0.07+collision_model_enlargement*2} ${0.03+collision_model_enlargement*2} ${0.022+collision_model_enlargement*2}"/>
+          </geometry>
+        </collision>
+      </xacro:if>
+      <!-- collision mesh used for grasp planning -->
+      <xacro:if value="$(arg collision_model_full)">
+        <collision>
+          <origin xyz="0 0 0" rpy="${PI} ${0.5 * PI} 0" />
+          <geometry>
+            <mesh filename="${homeDirectory}/meshes/secondFingerLink.stl"/>
+          </geometry>
+        </collision>
+      </xacro:if>
+      </xacro:unless>
+    </link>
+    <gazebo reference="${prefix}_HandFinger${number}KnuckleTwoLink">
+      <turnGravityOff>true</turnGravityOff>
+    </gazebo>
+    <joint name="${prefix}_HandFinger${number}KnuckleTwoJoint" type="revolute">
+      <parent link="${parent}"/>
+      <child link="${prefix}_HandFinger${number}KnuckleTwoLink"/>
+      <origin xyz="${xyz}" rpy="${rpy}"/>
+      <axis xyz="0 0 -1"/>
+                      <!-- 122 degrees - start orientation of 0.4 degrees-->
+      <limit effort="1" lower="0" upper="2.443388889" velocity="3.27"/>
+      <dynamics damping="0.005" friction="100.0"/>
+    </joint>
+  </xacro:macro>
+  <xacro:macro name="KnuckleThree" params="prefix number">
+    <link name="${prefix}_HandFinger${number}KnuckleThreeLink">
+      <visual>
+        <origin xyz="0 0 0" rpy="0 ${0.5 * PI} 0" />
+        <geometry>
+          <mesh filename="${homeDirectory}/meshes/KnuckleThreeLink.dae"/>
+        </geometry>
+      </visual>
+      <inertial>
+        <origin xyz="0.01970974 0.00182016 0.00020041" />
+        <mass value="0.03421781" />
+        <inertia  ixx="0.00000287" ixy="0.00000091"  ixz="-0.00000007"
+                                   iyy="0.00001329"  iyz="-0.00000002"
+                                                     izz="0.00001214" />
+      </inertial>
+      <xacro:unless value="$(arg collision_model_no_hands)">
+      <!-- collision mesh used for whole arm motion planning -->
+      <xacro:if value="$(arg collision_model_simplified)">
+        <collision>
+          <origin xyz="0.025 0 0" rpy="0 0 0" />
+          <geometry>
+            <box size="${0.07+collision_model_enlargement*2} ${0.02+collision_model_enlargement*2} ${0.022+collision_model_enlargement*2}"/>
+          </geometry>
+        </collision>
+      </xacro:if>
+      <!-- collision mesh used for grasp planning -->
+      <xacro:if value="$(arg collision_model_full)">
+        <collision>
+          <origin xyz="0 0 0" rpy="0 ${0.5 * PI} 0" />
+          <geometry>
+            <mesh filename="${homeDirectory}/meshes/thirdFingerLink.stl"/>
+          </geometry>
+        </collision>
+      </xacro:if>
+      </xacro:unless>
+    </link>
+    <gazebo reference="${prefix}_HandFinger${number}KnuckleThreeLink">
+      <turnGravityOff>true</turnGravityOff>
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