Commit message: self-collision model

File: barrett_hand_defs/defs/barret_hand.urdf.xacro (robot description, xacro)
@@ -77,18 +77,16 @@
       </xacro:unless>
       <!-- collision mesh used for RT self-collision avoidance -->
+<!--
       <self_collision_checking>
         <origin xyz="0 0 0" rpy="0 0 0"/>
         <geometry>
           <convex>
-            <!-- gripper base points -->
             <point xyz="0.03 0.03 0.0" frame="${prefix}_HandPalmLink"/>
             <point xyz="-0.03 0.03 0.0" frame="${prefix}_HandPalmLink"/>
             <point xyz="-0.03 -0.03 0.0" frame="${prefix}_HandPalmLink"/>
             <point xyz="0.03 -0.03 0.0" frame="${prefix}_HandPalmLink"/>
-            <!-- fingers' base links -->
             <point xyz="0.06 0 0" frame="${prefix}_HandFingerOneKnuckleOneLink"/>
             <point xyz="0.06 0 0" frame="${prefix}_HandFingerTwoKnuckleOneLink"/>
             <point xyz="0 -0.06 0.06" frame="${prefix}_HandPalmLink"/>
-            <!-- distal fingers' links -->
             <point xyz="0 0 0" frame="${prefix}_HandFingerOneKnuckleThreeLink"/>
             <point xyz="0 0 0" frame="${prefix}_HandFingerTwoKnuckleThreeLink"/>
@@ -100,4 +98,11 @@
         </geometry>
       </self_collision_checking>
+-->
+      <self_collision_checking>
+        <origin xyz="0.0 0.0 0.04" rpy="0 0 0"/>
+        <geometry>
+          <sphere radius="0.06"/>
+        </geometry>
+      </self_collision_checking>
     </link>
     <gazebo reference="${prefix}_HandPalmLink">
@@ -194,4 +199,10 @@
       </xacro:if>
       </xacro:unless>
+      <self_collision_checking>
+        <origin xyz="0.04 -0.01 0.0" rpy="0 1.57075 -0.5"/>
+        <geometry>
+          <capsule radius="0.03" length="0.1"/>
+        </geometry>
+      </self_collision_checking>
     </link>
     <gazebo reference="${prefix}_HandFinger${number}KnuckleTwoLink">

Commit message: added virtual link for gripper centre

File: barrett_hand_defs/defs/barret_hand.urdf.xacro (robot description, xacro)
@@ -115,4 +115,14 @@
       <provideFeedback value="true"/>
     </joint>
+    <link name="${prefix}_HandGripLink" >
+    </link>
+    <gazebo reference="${prefix}_HandGripLink">
+      <turnGravityOff>true</turnGravityOff>
+    </gazebo>
+    <joint name="${prefix}_HandGripJoint" type="fixed">
+      <parent link="${prefix}_HandPalmLink"/>
+      <child link="${prefix}_HandGripLink"/>
+      <origin rpy="0 0 0" xyz="0 0 0.12"/>
+    </joint>
   </xacro:macro>
   <xacro:macro name="KnuckleOne" params="prefix number xyz rpy axis">

Commit message: bugs in the urdf

File: barrett_hand_defs/defs/barret_hand.urdf.xacro (robot description, xacro)
@@ -155,5 +155,5 @@
       <xacro:if value="$(arg collision_model_full)">
         <collision>
-          <origin xyz="0 0 0" rpy="${0.5 * PI} 0 -${0.5 * PI}" />
+          <origin xyz="0 0 -0.0045" rpy="${0.5 * PI} 0 -${0.5 * PI}" />
           <geometry>
             <mesh filename="${homeDirectory}/meshes/firstFingerLink.stl"/>

Commit message: collision model

File: barrett_hand_defs/defs/barret_hand.urdf.xacro (robot description, xacro)
@@ -211,4 +211,11 @@
       </xacro:unless>
       <self_collision_checking>
+        <origin xyz="0.03 0.0 0.0" rpy="0 1.57075 0"/>
+        <geometry>
+          <capsule radius="0.01" length="0.06"/>
+        </geometry>
+      </self_collision_checking>
+<!--
+      <self_collision_checking>
         <origin xyz="0.04 -0.01 0.0" rpy="0 1.57075 -0.5"/>
         <geometry>
@@ -216,4 +223,5 @@
         </geometry>
       </self_collision_checking>
+-->
     </link>
     <gazebo reference="${prefix}_HandFinger${number}KnuckleTwoLink">
@@ -265,4 +273,10 @@
       </xacro:if>
       </xacro:unless>
+      <self_collision_checking>
+        <origin xyz="0.025 0.0 0.0" rpy="0 1.57075 0"/>
+        <geometry>
+          <capsule radius="0.0075" length="0.05"/>
+        </geometry>
+      </self_collision_checking>
     </link>
     <gazebo reference="${prefix}_HandFinger${number}KnuckleThreeLink">

Commit message: collision model for palm

File: barrett_hand_defs/defs/barret_hand.urdf.xacro (robot description, xacro)
@@ -101,5 +101,5 @@
 -->
       <self_collision_checking>
-        <origin xyz="0.0 0.0 0.04" rpy="0 0 0"/>
+        <origin xyz="0.0 0.0 0.02" rpy="0 0 0"/>
         <geometry>
           <sphere radius="0.06"/>

Commit message: added BH model with Optoforce sensors

File: barrett_hand_defs/defs/barret_hand.urdf.xacro (robot description, xacro)
@@ -32,8 +32,15 @@
   <xacro:arg name="collision_model_enlargement" default="0.0"/>
   <xacro:arg name="collision_model_no_hands" default="false"/>
+  <xacro:arg name="optoforce" default="false" />
   <xacro:property name="homeDirectory" value="package://barrett_hand_defs" />
   <xacro:property name="highResModelDirectory" value="${homeDirectory}/meshes/splitModels" />
   <xacro:property name="PI" value="3.1415926535897931" />
   <property name="collision_model_enlargement" value="$(arg collision_model_enlargement)" />
+  <xacro:if value="$(arg optoforce)">
+    <property name="optoforce" value="$(arg optoforce)" />
+  </xacro:if>
+  <xacro:unless value="$(arg optoforce)">
+    <property name="optoforce" value="" />
+  </xacro:unless>
   <xacro:macro name="palm" params="prefix parent *origin">
     <link name="${prefix}_HandPalmLink" >
@@ -243,5 +250,5 @@
         <origin xyz="0 0 0" rpy="0 ${0.5 * PI} 0" />
         <geometry>
-          <mesh filename="${homeDirectory}/meshes/KnuckleThreeLink.dae"/>
+          <mesh filename="${homeDirectory}/meshes/KnuckleThree${optoforce}Link.dae"/>
         </geometry>
       </visual>
@@ -268,5 +275,5 @@
           <origin xyz="0 0 0" rpy="0 ${0.5 * PI} 0" />
           <geometry>
-            <mesh filename="${homeDirectory}/meshes/thirdFingerLink.stl"/>
+            <mesh filename="${homeDirectory}/meshes/thirdFinger${optoforce}Link.stl"/>
           </geometry>
         </collision>
@@ -293,4 +300,20 @@
       <dynamics damping="0.005" friction="100.0"/>
     </joint>
+    <xacro:if value="$(arg optoforce)">
+        <link name="${prefix}_HandFinger${number}KnuckleThreeOptoforceBase" >
+        </link>
+        <joint name="${prefix}_HandFinger${number}KnuckleThreeOptoforceBaseJoint" type="fixed">
+          <parent link="${prefix}_HandFinger${number}KnuckleThreeLink"/>
+          <child link="${prefix}_HandFinger${number}KnuckleThreeOptoforceBase"/>
+          <origin rpy="0 0 -${35.0 * PI / 180.0}" xyz="0.0415 -0.0045 0"/>
+        </joint>
+        <link name="${prefix}_HandFinger${number}KnuckleThreeOptoforce" >
+        </link>
+        <joint name="${prefix}_HandFinger${number}KnuckleThreeOptoforceJoint" type="fixed">
+          <parent link="${prefix}_HandFinger${number}KnuckleThreeOptoforceBase"/>
+          <child link="${prefix}_HandFinger${number}KnuckleThreeOptoforce"/>
+          <origin rpy="0 ${PI/2} 0" xyz="0.005 0 0"/>
+        </joint>
+    </xacro:if>
   </xacro:macro>
   <xacro:macro name="fingers" params="parent prefix number xyz rpy">

Commit message: removed unnecessary friction from urdf joints

File: barrett_hand_defs/defs/barret_hand.urdf.xacro (robot description, xacro)
@@ -179,5 +179,5 @@
       <axis xyz="${axis}"/>
       <limit effort="1" lower="0" upper="${PI}" velocity="3.27"/>
-      <dynamics damping="0.05" friction="100.0"/>
+      <dynamics damping="0.05"/>
     </joint>
   </xacro:macro>
@@ -242,5 +242,5 @@
                       <!-- 122 degrees - start orientation of 0.4 degrees-->
       <limit effort="1" lower="0" upper="2.443388889" velocity="3.27"/>
-      <dynamics damping="0.005" friction="100.0"/>
+      <dynamics damping="0.005"/>
     </joint>
   </xacro:macro>
@@ -298,5 +298,5 @@
                           <!-- measured max angle is 94.  so upper limit is 94 - start orientation (42 degrees)-->
       <limit effort="1" lower="0" upper="0.837733333" velocity="3.27"/>
-      <dynamics damping="0.005" friction="100.0"/>
+      <dynamics damping="0.005"/>
     </joint>
     <xacro:if value="$(arg optoforce)">

Commit message: greater joint damping

File: barrett_hand_defs/defs/barret_hand.urdf.xacro (robot description, xacro)
@@ -179,5 +179,5 @@
       <axis xyz="${axis}"/>
       <limit effort="1" lower="0" upper="${PI}" velocity="3.27"/>
-      <dynamics damping="0.05"/>
+      <dynamics damping="0.1"/>
     </joint>
   </xacro:macro>
@@ -242,5 +242,5 @@
                       <!-- 122 degrees - start orientation of 0.4 degrees-->
       <limit effort="1" lower="0" upper="2.443388889" velocity="3.27"/>
-      <dynamics damping="0.005"/>
+      <dynamics damping="0.05"/>
     </joint>
   </xacro:macro>
@@ -298,5 +298,5 @@
                           <!-- measured max angle is 94.  so upper limit is 94 - start orientation (42 degrees)-->
       <limit effort="1" lower="0" upper="0.837733333" velocity="3.27"/>
-      <dynamics damping="0.005"/>
+      <dynamics damping="0.05"/>
     </joint>
     <xacro:if value="$(arg optoforce)">

Commit message: better Optoforce swith in urdf files

File: barrett_hand_defs/defs/barret_hand.urdf.xacro (robot description, xacro)
@@ -32,9 +32,9 @@
   <xacro:arg name="collision_model_enlargement" default="0.0"/>
   <xacro:arg name="collision_model_no_hands" default="false"/>
-  <xacro:arg name="optoforce" default="false" />
   <xacro:property name="homeDirectory" value="package://barrett_hand_defs" />
   <xacro:property name="highResModelDirectory" value="${homeDirectory}/meshes/splitModels" />
   <xacro:property name="PI" value="3.1415926535897931" />
   <property name="collision_model_enlargement" value="$(arg collision_model_enlargement)" />
+<!--
   <xacro:if value="$(arg optoforce)">
     <property name="optoforce" value="$(arg optoforce)" />
@@ -43,4 +43,5 @@
     <property name="optoforce" value="" />
   </xacro:unless>
+-->
   <xacro:macro name="palm" params="prefix parent *origin">
     <link name="${prefix}_HandPalmLink" >
@@ -245,10 +246,15 @@
     </joint>
   </xacro:macro>
-  <xacro:macro name="KnuckleThree" params="prefix number">
+  <xacro:macro name="KnuckleThree" params="prefix number with_optoforce">
     <link name="${prefix}_HandFinger${number}KnuckleThreeLink">
       <visual>
         <origin xyz="0 0 0" rpy="0 ${0.5 * PI} 0" />
         <geometry>
-          <mesh filename="${homeDirectory}/meshes/KnuckleThree${optoforce}Link.dae"/>
+          <xacro:if value="${with_optoforce}">
+            <mesh filename="${homeDirectory}/meshes/KnuckleThreeOptoforceLink.dae"/>
+          </xacro:if>
+          <xacro:unless value="${with_optoforce}">
+            <mesh filename="${homeDirectory}/meshes/KnuckleThreeLink.dae"/>
+          </xacro:unless>
         </geometry>
       </visual>
@@ -275,5 +281,10 @@
           <origin xyz="0 0 0" rpy="0 ${0.5 * PI} 0" />
           <geometry>
-            <mesh filename="${homeDirectory}/meshes/thirdFinger${optoforce}Link.stl"/>
+            <xacro:if value="${with_optoforce}">
+              <mesh filename="${homeDirectory}/meshes/thirdFingerOptoforceLink.stl"/>
+            </xacro:if>
+            <xacro:unless value="${with_optoforce}">
+              <mesh filename="${homeDirectory}/meshes/thirdFingerLink.stl"/>
+            </xacro:unless>
           </geometry>
         </collision>
@@ -300,5 +311,5 @@
       <dynamics damping="0.05"/>
     </joint>
-    <xacro:if value="$(arg optoforce)">
+    <xacro:if value="${with_optoforce}">
         <link name="${prefix}_HandFinger${number}KnuckleThreeOptoforceBase" >
         </link>
@@ -317,17 +328,17 @@
     </xacro:if>
   </xacro:macro>
-  <xacro:macro name="fingers" params="parent prefix number xyz rpy">
+  <xacro:macro name="fingers" params="parent prefix number xyz rpy with_optoforce">
     <xacro:KnuckleTwo parent="${parent}" prefix="${prefix}" number="${number}" xyz="${xyz}" rpy="${rpy}" />
-    <xacro:KnuckleThree prefix="${prefix}" number="${number}"/>
-  </xacro:macro>
-    <xacro:macro name="barret_hand" params="prefix parent *origin">
+    <xacro:KnuckleThree prefix="${prefix}" number="${number}" with_optoforce="${with_optoforce}"/>
+  </xacro:macro>
+    <xacro:macro name="barret_hand" params="prefix parent *origin with_optoforce">
         <xacro:palm prefix="${prefix}" parent="${parent}">
             <insert_block name="origin"/>
         </xacro:palm>
-        <xacro:fingers prefix="${prefix}" parent="${prefix}_HandPalmLink" number="Three" xyz="0 -0.05 0.0754" rpy="-${0.5 * PI} 0 -${0.5 * PI}"/>
+        <xacro:fingers prefix="${prefix}" parent="${prefix}_HandPalmLink" number="Three" xyz="0 -0.05 0.0754" rpy="-${0.5 * PI} 0 -${0.5 * PI}" with_optoforce="${with_optoforce}"/>
         <xacro:KnuckleOne prefix="${prefix}" number="One" xyz=".02497 0 0.0587966" rpy="0 0 ${0.5 * PI}" axis="0 0 -1"/>
-        <xacro:fingers prefix="${prefix}" parent="${prefix}_HandFingerOneKnuckleOneLink" number="One" xyz=".05 0 0.0166034" rpy="-${0.5 * PI} 0 0"/>
+        <xacro:fingers prefix="${prefix}" parent="${prefix}_HandFingerOneKnuckleOneLink" number="One" xyz=".05 0 0.0166034" rpy="-${0.5 * PI} 0 0" with_optoforce="${with_optoforce}"/>
         <xacro:KnuckleOne prefix="${prefix}" number="Two" xyz="-.02497 0 0.0587966" rpy="0 0 ${0.5 * PI}" axis ="0 0 1"/>
-        <xacro:fingers prefix="${prefix}" parent="${prefix}_HandFingerTwoKnuckleOneLink" number="Two" xyz=".05 0 0.0166034" rpy="-${0.5 * PI} 0 0"/>
+        <xacro:fingers prefix="${prefix}" parent="${prefix}_HandFingerTwoKnuckleOneLink" number="Two" xyz=".05 0 0.0166034" rpy="-${0.5 * PI} 0 0" with_optoforce="${with_optoforce}"/>
 <!--        <xacro:fingers prefix="${prefix}" parent="${prefix}_HandFingerTwoKnuckleOneLink" number="Two" xyz=".05 0 0.0166034" rpy="-${0.5 * PI} -0.0429350996 0"/>-->
 </xacro:macro>

Commit message: zero rotation for distal finger link collision geometry

File: barrett_hand_defs/defs/barret_hand.urdf.xacro (robot description, xacro)
@@ -271,5 +271,5 @@
       <xacro:if value="$(arg collision_model_full)">
         <collision>
-          <origin xyz="0 0 0" rpy="0 ${0.5 * PI} 0" />
+          <origin xyz="0 0 0" rpy="0 0 0" />
           <geometry>
             <xacro:if value="${with_optoforce}">

Commit message: optoforce sensors

File: barrett_hand_defs/defs/barret_hand.urdf.xacro (robot description, xacro)
@@ -244,5 +244,5 @@
         <geometry>
           <xacro:if value="${with_optoforce}">
-            <mesh filename="${homeDirectory}/meshes/KnuckleThreeOptoforceLink.dae"/>
+            <mesh filename="${homeDirectory}/meshes/KnuckleThreeOptoforceBaseLink.dae"/>
           </xacro:if>
           <xacro:unless value="${with_optoforce}">
@@ -274,5 +274,5 @@
           <geometry>
             <xacro:if value="${with_optoforce}">
-              <mesh filename="${homeDirectory}/meshes/thirdFingerOptoforceLink.stl"/>
+              <mesh filename="${homeDirectory}/meshes/thirdFingerOptoforceBaseLink.stl"/>
             </xacro:if>
             <xacro:unless value="${with_optoforce}">
@@ -304,4 +304,47 @@
     </joint>
     <xacro:if value="${with_optoforce}">
+        <link name="${prefix}_HandFinger${number}KnuckleThreeOptoforceBase" >
+          <visual>
+            <origin xyz="0 0 0" rpy="0 0 0" />
+            <geometry>
+              <sphere radius="0.01"/>
+            </geometry>
+          </visual>
+        </link>
+        <joint name="${prefix}_HandFinger${number}KnuckleThreeOptoforceBaseJoint" type="fixed">
+          <parent link="${prefix}_HandFinger${number}KnuckleThreeLink"/>
+          <child link="${prefix}_HandFinger${number}KnuckleThreeOptoforceBase"/>
+          <origin rpy="0 ${PI/2} -${35.0 * PI / 180.0}" xyz="0.04486 -0.00685 0"/>
+        </joint>
+        <gazebo reference="${prefix}_HandFinger${number}KnuckleThreeOptoforceBase">
+          <turnGravityOff>true</turnGravityOff>
+        </gazebo>
+        <link name="${prefix}_HandFinger${number}KnuckleThreeOptoforceSensor" >
+          <inertial>
+            <origin xyz="0 0 0" />
+            <mass value="0.003421781" />
+            <inertia  ixx="0.000000287" ixy="0.000000091"  ixz="-0.000000007"
+                                         iyy="0.000001329"  iyz="-0.000000002"
+                                                             izz="0.000001214" />
+          </inertial>
+          <collision>
+            <origin xyz="0 0 0" rpy="0 0 0" />
+            <geometry>
+              <sphere radius="0.01"/>
+            </geometry>
+          </collision>
+        </link>
+        <joint name="${prefix}_HandFinger${number}KnuckleThreeOptoforceJoint" type="prismatic">
+          <parent link="${prefix}_HandFinger${number}KnuckleThreeLink"/>
+          <child link="${prefix}_HandFinger${number}KnuckleThreeOptoforceSensor"/>
+          <origin rpy="0 ${PI/2} -${35.0 * PI / 180.0}" xyz="0.04486 -0.00685 0"/>
+          <axis xyz="0 0 1"/>
+          <limit effort="2" lower="-0.005" upper="0.005" velocity="0.1"/>
+          <dynamics damping="0.1"/>
+        </joint>
+        <gazebo reference="${prefix}_HandFinger${number}KnuckleThreeOptoforceSensor">
+          <turnGravityOff>true</turnGravityOff>
+        </gazebo>
+<!--
         <link name="${prefix}_HandFinger${number}KnuckleThreeOptoforceBase" >
         </link>
@@ -318,4 +361,5 @@
           <origin rpy="0 ${PI/2} 0" xyz="0.005 0 0"/>
         </joint>
+-->
     </xacro:if>
   </xacro:macro>

Commit message: valid inertia matrix

File: barrett_hand_defs/defs/barret_hand.urdf.xacro (robot description, xacro)
@@ -251,5 +251,5 @@
         </geometry>
       </visual>
-      <inertial>
+<!--      <inertial>
         <origin xyz="0.01970974 0.00182016 0.00020041" />
         <mass value="0.03421781" />
@@ -257,4 +257,12 @@
                                    iyy="0.00001329"  iyz="-0.00000002"
                                                      izz="0.00001214" />
+      </inertial>
+-->
+      <inertial>
+        <origin xyz=".031720 .001070 -.000586" />
+        <mass value="0.057957" />
+        <inertia  ixx="0.00000461" ixy="0.00000003"  ixz="0.00000164"
+                                   iyy="0.00003590"  iyz="0.00000004"
+                                                     izz="0.00003682" />
       </inertial>
       <xacro:unless value="$(arg collision_model_no_hands)">

Commit message: inertia matrix for knuckle 3

File: barrett_hand_defs/defs/barret_hand.urdf.xacro (robot description, xacro)
@@ -266,6 +266,6 @@
 -->
       <inertial>
-        <origin xyz=".031720 .001070 -.000586" />
-        <mass value="0.057957" />
+        <origin xyz="0.01970974 0.00182016 0.00020041" />
+        <mass value="0.03421781" />
         <inertia  ixx="0.00000461" ixy="0.00000003"  ixz="0.00000164"
                                    iyy="0.00003590"  iyz="0.00000004"

Commit message: added material for optoforce ball

File: barrett_hand_defs/defs/barret_hand.urdf.xacro (robot description, xacro)
@@ -327,4 +327,7 @@
               <sphere radius="0.01"/>
             </geometry>
+            <material name="material_optoforce_ball">
+              <color rgba="0.7 0.7 0.7 1.0"/>
+            </material>
           </visual>
         </link>

Commit message: better colors for barrethand

File: barrett_hand_defs/defs/barret_hand.urdf.xacro (robot description, xacro)
@@ -28,4 +28,5 @@
        xmlns:interface="http://playerstage.sourceforge.net/gazebo/xmlschema/#interface"
        xmlns:xacro="http://www.ros.org/wiki/xacro">
+  <xacro:include filename="$(find barrett_hand_defs)/defs/materials.xml"/>
   <xacro:arg name="collision_model_full" default="true"/>
   <xacro:arg name="collision_model_simplified" default="false"/>
@@ -50,4 +51,5 @@
           <mesh filename="${homeDirectory}/meshes/HandPalmLink.dae"/>
         </geometry>
+        <material name="bh_HandGrey"/>
       </visual>
       <xacro:unless value="$(arg collision_model_no_hands)">
@@ -134,4 +136,5 @@
           <mesh filename="${homeDirectory}/meshes/KnuckleOneLink.dae"/>
         </geometry>
+        <material name="bh_HandGrey"/>
       </visual>
       <inertial>
@@ -185,4 +188,5 @@
           <mesh filename="${homeDirectory}/meshes/KnuckleTwoLink.dae"/>
         </geometry>
+        <material name="bh_HandGrey"/>
       </visual>
       <inertial>
@@ -256,4 +260,5 @@
           </xacro:unless>
         </geometry>
+        <material name="bh_HandGrey"/>
       </visual>
 <!--      <inertial>
@@ -327,7 +332,5 @@
               <sphere radius="0.01"/>
             </geometry>
-            <material name="material_optoforce_ball">
-              <color rgba="0.7 0.7 0.7 1.0"/>
-            </material>
+            <material name="bh_Black"/>
           </visual>
         </link>

Commit message: wider collision objects for fingers

File: barrett_hand_defs/defs/barret_hand.urdf.xacro (robot description, xacro)
@@ -127,5 +127,5 @@
 -->
       <self_collision_checking>
-        <origin xyz="0.0 0.0 0.02" rpy="0 0 0"/>
+        <origin xyz="0.0 0.0 0.03" rpy="0 0 0"/>
         <geometry>
           <sphere radius="0.06"/>
@@ -279,5 +279,5 @@
         <origin xyz="0.03 0.0 0.0" rpy="0 1.57075 0"/>
         <geometry>
-          <capsule radius="0.01" length="0.06"/>
+          <capsule radius="0.015" length="0.06"/>
         </geometry>
       </self_collision_checking>
@@ -381,5 +381,5 @@
         <origin xyz="0.025 0.0 0.0" rpy="0 1.57075 0"/>
         <geometry>
-          <capsule radius="0.0075" length="0.05"/>
+          <capsule radius="0.015" length="0.05"/>
         </geometry>
       </self_collision_checking>
