Commit message: simplified visual model

File: barrett_hand_defs/defs/barret_hand.urdf.xacro (robot description, xacro)
@@ -47,7 +47,7 @@
       </inertial>
       <visual>
-        <origin xyz="0 0 0" rpy="${PI} 0 0" />
-        <geometry>
-          <mesh filename="${homeDirectory}/meshes/HandPalmLink.dae"/>
+        <origin xyz="0 0 0" rpy="0 0 0" />
+        <geometry>
+          <mesh filename="${homeDirectory}/meshes/palm.stl"/>
         </geometry>
         <material name="bh_HandGrey"/>
@@ -158,7 +158,7 @@
     <link name="${prefix}_HandFinger${number}KnuckleOneLink">
       <visual>
-        <origin xyz="0 0 -0.017" rpy="${0.5 * PI} 0 -${0.5 * PI}" />
-        <geometry>
-          <mesh filename="${homeDirectory}/meshes/KnuckleOneLink.dae"/>
+        <origin xyz="0 0 -0.0045" rpy="${0.5 * PI} 0 -${0.5 * PI}" />
+        <geometry>
+          <mesh filename="${homeDirectory}/meshes/firstFingerLink.stl"/>
         </geometry>
         <material name="bh_HandGrey"/>
@@ -229,5 +229,5 @@
         <origin xyz="0 0 0" rpy="${PI} ${0.5 * PI} 0" />
         <geometry>
-          <mesh filename="${homeDirectory}/meshes/KnuckleTwoLink.dae"/>
+          <mesh filename="${homeDirectory}/meshes/secondFingerLink.stl"/>
         </geometry>
         <material name="bh_HandGrey"/>
@@ -311,11 +311,11 @@
     <link name="${prefix}_HandFinger${number}KnuckleThreeLink">
       <visual>
-        <origin xyz="0 0 0" rpy="0 ${0.5 * PI} 0" />
+        <origin xyz="0 0 0" rpy="0 0 0" />
         <geometry>
           <xacro:if value="${with_optoforce}">
-            <mesh filename="${homeDirectory}/meshes/KnuckleThreeOptoforceBaseLink.dae"/>
+            <mesh filename="${homeDirectory}/meshes/thirdFingerOptoforceBaseLink.stl"/>
           </xacro:if>
           <xacro:unless value="${with_optoforce}">
-            <mesh filename="${homeDirectory}/meshes/KnuckleThreeLink.dae"/>
+            <mesh filename="${homeDirectory}/meshes/thirdFingerLink.stl"/>
           </xacro:unless>
         </geometry>

Commit message: fix XACROs for ROS Melodic

File: barrett_hand_defs/defs/barret_hand.urdf.xacro (robot description, xacro)
@@ -92,18 +92,17 @@
             <mesh filename="${homeDirectory}/meshes/palm.stl"/>
           </geometry>
-            <surface>
-              <friction>
-                <ode>
-                  <mu>1.0</mu>
-                  <mu2>1.0</mu2>
-                </ode>
-              </friction>
-            </surface>
+          <surface>
+            <friction>
+              <ode>
+                <mu>1.0</mu>
+                <mu2>1.0</mu2>
+              </ode>
+            </friction>
+          </surface>
         </collision>
       </xacro:if>
       </xacro:unless>
       <!-- collision mesh used for RT self-collision avoidance -->
-<!--
-      <self_collision_checking>
+      <!-- <self_collision_checking>
         <origin xyz="0 0 0" rpy="0 0 0"/>
         <geometry>
@@ -124,6 +123,5 @@
           </convex>
         </geometry>
-      </self_collision_checking>
--->
+      </self_collision_checking> -->
       <self_collision_checking>
         <origin xyz="0.0 0.0 0.03" rpy="0 0 0"/>
@@ -234,5 +232,5 @@
       </visual>
       <inertial>
-        <origin xyz=".031720 .001070 -.000586" />
+        <origin xyz="0.031720 0.001070 -0.000586" />
         <mass value="0.057957" />
         <inertia  ixx="0.00000461" ixy="0.00000003"  ixz="0.00000164"
@@ -480,14 +478,14 @@
     <xacro:KnuckleThree prefix="${prefix}" number="${number}" with_optoforce="${with_optoforce}"/>
   </xacro:macro>
-    <xacro:macro name="barret_hand" params="prefix parent *origin with_optoforce">
-        <xacro:palm prefix="${prefix}" parent="${parent}">
-            <insert_block name="origin"/>
-        </xacro:palm>
-        <xacro:fingers prefix="${prefix}" parent="${prefix}_HandPalmLink" number="Three" xyz="0 -0.05 0.0754" rpy="-${0.5 * PI} 0 -${0.5 * PI}" with_optoforce="${with_optoforce}"/>
-        <xacro:KnuckleOne prefix="${prefix}" number="One" xyz=".02497 0 0.0587966" rpy="0 0 ${0.5 * PI}" axis="0 0 -1"/>
-        <xacro:fingers prefix="${prefix}" parent="${prefix}_HandFingerOneKnuckleOneLink" number="One" xyz=".05 0 0.0166034" rpy="-${0.5 * PI} 0 0" with_optoforce="${with_optoforce}"/>
-        <xacro:KnuckleOne prefix="${prefix}" number="Two" xyz="-.02497 0 0.0587966" rpy="0 0 ${0.5 * PI}" axis ="0 0 1"/>
-        <xacro:fingers prefix="${prefix}" parent="${prefix}_HandFingerTwoKnuckleOneLink" number="Two" xyz=".05 0 0.0166034" rpy="-${0.5 * PI} 0 0" with_optoforce="${with_optoforce}"/>
-<!--        <xacro:fingers prefix="${prefix}" parent="${prefix}_HandFingerTwoKnuckleOneLink" number="Two" xyz=".05 0 0.0166034" rpy="-${0.5 * PI} -0.0429350996 0"/>-->
-</xacro:macro>
+  <xacro:macro name="barret_hand" params="prefix parent *origin with_optoforce">
+    <xacro:palm prefix="${prefix}" parent="${parent}">
+      <insert_block name="origin"/>
+    </xacro:palm>
+    <xacro:fingers prefix="${prefix}" parent="${prefix}_HandPalmLink" number="Three" xyz="0 -0.05 0.0754" rpy="-${0.5 * PI} 0 -${0.5 * PI}" with_optoforce="${with_optoforce}"/>
+    <xacro:KnuckleOne prefix="${prefix}" number="One" xyz="0.02497 0 0.0587966" rpy="0 0 ${0.5 * PI}" axis="0 0 -1"/>
+    <xacro:fingers prefix="${prefix}" parent="${prefix}_HandFingerOneKnuckleOneLink" number="One" xyz="0.05 0 0.0166034" rpy="-${0.5 * PI} 0 0" with_optoforce="${with_optoforce}"/>
+    <xacro:KnuckleOne prefix="${prefix}" number="Two" xyz="-0.02497 0 0.0587966" rpy="0 0 ${0.5 * PI}" axis ="0 0 1"/>
+    <xacro:fingers prefix="${prefix}" parent="${prefix}_HandFingerTwoKnuckleOneLink" number="Two" xyz="0.05 0 0.0166034" rpy="-${0.5 * PI} 0 0" with_optoforce="${with_optoforce}"/>
+    <!-- <xacro:fingers prefix="${prefix}" parent="${prefix}_HandFingerTwoKnuckleOneLink" number="Two" xyz="0.05 0 0.0166034" rpy="-${0.5 * PI} -0.0429350996 0"/> -->
+  </xacro:macro>
 </robot>

File: barrett_hand_defs/defs/barret_hand_export.urdf.xacro (robot description, xacro)
@@ -133,5 +133,5 @@
             </visual>
             <inertial>
-                <origin xyz=".031720 .001070 -.000586" />
+                <origin xyz="0.031720 0.001070 -0.000586" />
                 <mass value="0.057957" />
                 <inertia  ixx="0.00000461" ixy="0.00000003"  ixz="0.00000164"
@@ -212,9 +212,9 @@
         </xacro:palm>
         <xacro:fingers prefix="${prefix}" parent="${prefix}_HandPalmLink" number="Three" xyz="0 -0.05 0.0754" rpy="-${0.5 * PI} 0 -${0.5 * PI}"/>
-        <xacro:KnuckleOne prefix="${prefix}" number="One" xyz=".02497 0 0.0587966" rpy="0 0 ${0.5 * PI}" axis="0 0 -1"/>
-        <xacro:fingers prefix="${prefix}" parent="${prefix}_HandFingerOneKnuckleOneLink" number="One" xyz=".05 0 0.0166034" rpy="-${0.5 * PI} 0 0"/>
-        <xacro:KnuckleOne prefix="${prefix}" number="Two" xyz="-.02497 0 0.0587966" rpy="0 0 ${0.5 * PI}" axis ="0 0 1"/>
-        <xacro:fingers prefix="${prefix}" parent="${prefix}_HandFingerTwoKnuckleOneLink" number="Two" xyz=".05 0 0.0166034" rpy="-${0.5 * PI} 0 0"/>
-<!--        <xacro:fingers prefix="${prefix}" parent="${prefix}_HandFingerTwoKnuckleOneLink" number="Two" xyz=".05 0 0.0166034" rpy="-${0.5 * PI} -0.0429350996 0"/>-->
+        <xacro:KnuckleOne prefix="${prefix}" number="One" xyz="0.02497 0 0.0587966" rpy="0 0 ${0.5 * PI}" axis="0 0 -1"/>
+        <xacro:fingers prefix="${prefix}" parent="${prefix}_HandFingerOneKnuckleOneLink" number="One" xyz="0.05 0 0.0166034" rpy="-${0.5 * PI} 0 0"/>
+        <xacro:KnuckleOne prefix="${prefix}" number="Two" xyz="-0.02497 0 0.0587966" rpy="0 0 ${0.5 * PI}" axis ="0 0 1"/>
+        <xacro:fingers prefix="${prefix}" parent="${prefix}_HandFingerTwoKnuckleOneLink" number="Two" xyz="0.05 0 0.0166034" rpy="-${0.5 * PI} 0 0"/>
+<!--        <xacro:fingers prefix="${prefix}" parent="${prefix}_HandFingerTwoKnuckleOneLink" number="Two" xyz="0.05 0 0.0166034" rpy="-${0.5 * PI} -0.0429350996 0"/>-->
 </xacro:macro>
 </robot>

Commit message: improved visualization of optoforce sensors

File: barrett_hand_defs/defs/barret_hand.urdf.xacro (robot description, xacro)
@@ -401,21 +401,4 @@
     </gazebo>
     <xacro:if value="${with_optoforce}">
-        <link name="${prefix}_HandFinger${number}KnuckleThreeOptoforceBase" >
-          <visual>
-            <origin xyz="0 0 0" rpy="0 0 0" />
-            <geometry>
-              <sphere radius="0.01"/>
-            </geometry>
-            <material name="bh_Black"/>
-          </visual>
-        </link>
-        <joint name="${prefix}_HandFinger${number}KnuckleThreeOptoforceBaseJoint" type="fixed">
-          <parent link="${prefix}_HandFinger${number}KnuckleThreeLink"/>
-          <child link="${prefix}_HandFinger${number}KnuckleThreeOptoforceBase"/>
-          <origin rpy="0 ${PI/2} -${35.0 * PI / 180.0}" xyz="0.04486 -0.00685 0"/>
-        </joint>
-        <gazebo reference="${prefix}_HandFinger${number}KnuckleThreeOptoforceBase">
-          <turnGravityOff>false</turnGravityOff>
-        </gazebo>
         <link name="${prefix}_HandFinger${number}KnuckleThreeOptoforceSensor" >
           <inertial>
@@ -426,4 +409,11 @@
                                                              izz="0.000001214" />
           </inertial>
+          <visual>
+            <origin xyz="0 0 0" rpy="0 0 0" />
+            <geometry>
+              <sphere radius="0.01"/>
+            </geometry>
+            <material name="bh_Black"/>
+          </visual>
           <collision>
             <origin xyz="0 0 0" rpy="0 0 0" />
@@ -456,20 +446,4 @@
           <selfCollide>true</selfCollide>
         </gazebo>
-<!--
-        <link name="${prefix}_HandFinger${number}KnuckleThreeOptoforceBase" >
-        </link>
-        <joint name="${prefix}_HandFinger${number}KnuckleThreeOptoforceBaseJoint" type="fixed">
-          <parent link="${prefix}_HandFinger${number}KnuckleThreeLink"/>
-          <child link="${prefix}_HandFinger${number}KnuckleThreeOptoforceBase"/>
-          <origin rpy="0 0 -${35.0 * PI / 180.0}" xyz="0.0415 -0.0045 0"/>
-        </joint>
-        <link name="${prefix}_HandFinger${number}KnuckleThreeOptoforce" >
-        </link>
-        <joint name="${prefix}_HandFinger${number}KnuckleThreeOptoforceJoint" type="fixed">
-          <parent link="${prefix}_HandFinger${number}KnuckleThreeOptoforceBase"/>
-          <child link="${prefix}_HandFinger${number}KnuckleThreeOptoforce"/>
-          <origin rpy="0 ${PI/2} 0" xyz="0.005 0 0"/>
-        </joint>
--->
     </xacro:if>
   </xacro:macro>

Commit message: visual mesh for optoforce as stl mesh

File: barrett_hand_defs/defs/barret_hand.urdf.xacro (robot description, xacro)
@@ -412,5 +412,6 @@
             <origin xyz="0 0 0" rpy="0 0 0" />
             <geometry>
-              <sphere radius="0.01"/>
+              <mesh filename="${homeDirectory}/meshes/optoforce_sphere.stl"/>
+              <!--<sphere radius="0.01"/>-->
             </geometry>
             <material name="bh_Black"/>

Commit message: very simple collision geoms - fix for sticking objects in gazebo

File: barrett_hand_defs/defs/barret_hand.urdf.xacro (robot description, xacro)
@@ -259,7 +259,11 @@
       <xacro:if value="$(arg collision_model_full)">
         <collision>
-          <origin xyz="0 0 0" rpy="${PI} ${0.5 * PI} 0" />
+<!--          <origin xyz="0 0 0" rpy="${PI} ${0.5 * PI} 0" />
           <geometry>
             <mesh filename="${homeDirectory}/meshes/secondFingerLink.stl"/>
+          </geometry>-->
+          <origin xyz="0.03 0 0" rpy="0 0 0" />
+          <geometry>
+            <box size="0.07 0.02 0.02" />
           </geometry>
             <surface>
@@ -356,5 +360,5 @@
       <xacro:if value="$(arg collision_model_full)">
         <collision>
-          <origin xyz="0 0 0" rpy="0 0 0" />
+<!--          <origin xyz="0 0 0" rpy="0 0 0" />
           <geometry>
             <xacro:if value="${with_optoforce}">
@@ -364,4 +368,9 @@
               <mesh filename="${homeDirectory}/meshes/thirdFingerLink.stl"/>
             </xacro:unless>
+          </geometry>
+-->
+          <origin xyz="0.025 0 0" rpy="0 0 0" />
+          <geometry>
+            <box size="0.05 0.02 0.02" />
           </geometry>
             <surface>

Commit message: set mass to virtual link

File: barrett_hand_defs/defs/barret_hand.urdf.xacro (robot description, xacro)
@@ -143,4 +143,11 @@
     </joint>
     <link name="${prefix}_HandGripLink" >
+      <inertial>
+        <origin xyz="0.0 0.0 0.0" />
+        <mass value="0.005" />
+        <inertia  ixx="0.00000041" ixy="0.00000000"  ixz="0.00000016"
+                                   iyy="0.00000359"  iyz="0.00000000"
+                                                     izz="0.00000368" />
+      </inertial>
     </link>
     <gazebo reference="${prefix}_HandGripLink">

Commit message: increased limits for torque

File: barrett_hand_defs/defs/barret_hand.urdf.xacro (robot description, xacro)
@@ -223,5 +223,5 @@
       <origin xyz="${xyz}" rpy="${rpy}"/>
       <axis xyz="${axis}"/>
-      <limit effort="1" lower="0" upper="${PI}" velocity="3.27"/>
+      <limit effort="2" lower="0" upper="${PI}" velocity="3.27"/>
       <dynamics damping="0.1"/>
     </joint>
@@ -311,5 +311,5 @@
       <axis xyz="0 0 -1"/>
                       <!-- 122 degrees - start orientation of 0.4 degrees-->
-      <limit effort="1" lower="0" upper="2.443388889" velocity="3.27"/>
+      <limit effort="2" lower="0" upper="2.443388889" velocity="3.27"/>
       <dynamics damping="0.05"/>
     </joint>
@@ -411,5 +411,5 @@
       <axis xyz="0 0 -1"/>
                           <!-- measured max angle is 94.  so upper limit is 94 - start orientation (42 degrees)-->
-      <limit effort="1" lower="0" upper="0.837733333" velocity="3.27"/>
+      <limit effort="2" lower="0" upper="0.837733333" velocity="3.27"/>
       <dynamics damping="0.05"/>
     </joint>

Commit message: added marker a

File: barrett_hand_defs/defs/barret_hand.urdf.xacro (robot description, xacro)
@@ -136,4 +136,17 @@
       <selfCollide>true</selfCollide>
     </gazebo>
+    <joint name="${prefix}_HandPalmMarkerAJoint" type="fixed">
+      <parent link="${prefix}_HandPalmLink"/>
+      <child link="${prefix}_HandPalmMarkerALink"/>
+      <origin xyz="0.0445 0.0 0.0255" rpy="0 ${PI/2} 0" />
+    </joint>
+    <link name="${prefix}_HandPalmMarkerALink" >
+      <visual>
+        <origin xyz="0 0 0" rpy="0 0 0" />
+        <geometry>
+          <sphere radius="0.01"/>
+        </geometry>
+      </visual>
+    </link>
     <joint name="${prefix}_HandPalmJoint" type="fixed">
       <parent link="${parent}"/>

Commit message: added markers b,c,d

File: barrett_hand_defs/defs/barret_hand.urdf.xacro (robot description, xacro)
@@ -149,4 +149,43 @@
       </visual>
     </link>
+    <joint name="${prefix}_HandPalmMarkerCJoint" type="fixed">
+      <parent link="${prefix}_HandPalmLink"/>
+      <child link="${prefix}_HandPalmMarkerCLink"/>
+      <origin xyz="-0.0445 0.0 0.0255" rpy="0 ${-PI/2} 0" />
+    </joint>
+    <link name="${prefix}_HandPalmMarkerCLink" >
+      <visual>
+        <origin xyz="0 0 0" rpy="0 0 0" />
+        <geometry>
+          <sphere radius="0.01"/>
+        </geometry>
+      </visual>
+    </link>
+    <joint name="${prefix}_HandPalmMarkerBJoint" type="fixed">
+      <parent link="${prefix}_HandPalmLink"/>
+      <child link="${prefix}_HandPalmMarkerBLink"/>
+      <origin xyz="0.0 0.0445 0.0255" rpy="${-PI/2} 0 0" />
+    </joint>
+    <link name="${prefix}_HandPalmMarkerBLink" >
+      <visual>
+        <origin xyz="0 0 0" rpy="0 0 0" />
+        <geometry>
+          <sphere radius="0.01"/>
+        </geometry>
+      </visual>
+    </link>
+    <joint name="${prefix}_HandPalmMarkerDJoint" type="fixed">
+      <parent link="${prefix}_HandPalmLink"/>
+      <child link="${prefix}_HandPalmMarkerDLink"/>
+      <origin xyz="0.0 -0.0445 0.0255" rpy="${PI/2} 0 0" />
+    </joint>
+    <link name="${prefix}_HandPalmMarkerDLink" >
+      <visual>
+        <origin xyz="0 0 0" rpy="0 0 0" />
+        <geometry>
+          <sphere radius="0.01"/>
+        </geometry>
+      </visual>
+    </link>
     <joint name="${prefix}_HandPalmJoint" type="fixed">
       <parent link="${parent}"/>
