Commit message: dart collision model using spheres and boxes only

File: barrett_hand_defs/defs/barret_hand.urdf.xacro (robot description, xacro)
@@ -58,30 +58,26 @@
       <xacro:if value="$(arg collision_model_simplified)">
         <collision>
-          <origin xyz="0 0 0.045" rpy="0 0 0" />
-          <geometry>
-            <cylinder radius="${0.045+collision_model_enlargement}" length="0.09"/>
-          </geometry>
-            <surface>
-              <friction>
-                <ode>
-                  <mu>1.0</mu>
-                  <mu2>1.0</mu2>
-                </ode>
-              </friction>
-            </surface>
-        </collision>
-        <collision>
-          <origin xyz="0 -0.035 0.07" rpy="0 0 0" />
-          <geometry>
-            <box size="${0.025+collision_model_enlargement*2} ${0.08+collision_model_enlargement*2} ${0.05+collision_model_enlargement*2}"/>
-          </geometry>
-            <surface>
-              <friction>
-                <ode>
-                  <mu>1.0</mu>
-                  <mu2>1.0</mu2>
-                </ode>
-              </friction>
-            </surface>
+          <origin xyz="0 0 0.029" rpy="0 0 0"/>
+          <geometry>
+            <sphere radius="0.049"/>
+          </geometry>
+        </collision>
+        <collision>
+          <origin xyz="0 0 0.0578880161047" rpy="0 0 0"/>
+          <geometry>
+            <box size="0.0905260443687 0.0546207651496 0.0420634746552"/>
+          </geometry>
+        </collision>
+        <collision>
+          <origin xyz="0 -0.0385280400515 0.0572689175606" rpy="0 0 0"/>
+          <geometry>
+            <box size="0.0275810360909 0.0546207651496 0.0339374542236"/>
+          </geometry>
+        </collision>
+        <collision>
+          <origin xyz="0 -0.0487826019526 0.0744814276695" rpy="0 0 0"/>
+          <geometry>
+            <sphere radius="0.0194399058819"/>
+          </geometry>
         </collision>
       </xacro:if>
@@ -141,12 +137,5 @@
       <origin xyz="0.0445 0.0 0.0255" rpy="0 ${PI/2} 0" />
     </joint>
-    <link name="${prefix}_HandPalmMarkerALink" >
-      <visual>
-        <origin xyz="0 0 0" rpy="0 0 0" />
-        <geometry>
-          <sphere radius="0.01"/>
-        </geometry>
-      </visual>
-    </link>
+    <link name="${prefix}_HandPalmMarkerALink" />
     <joint name="${prefix}_HandPalmMarkerCJoint" type="fixed">
       <parent link="${prefix}_HandPalmLink"/>
@@ -154,12 +143,5 @@
       <origin xyz="-0.0445 0.0 0.0255" rpy="0 ${-PI/2} 0" />
     </joint>
-    <link name="${prefix}_HandPalmMarkerCLink" >
-      <visual>
-        <origin xyz="0 0 0" rpy="0 0 0" />
-        <geometry>
-          <sphere radius="0.01"/>
-        </geometry>
-      </visual>
-    </link>
+    <link name="${prefix}_HandPalmMarkerCLink" />
     <joint name="${prefix}_HandPalmMarkerBJoint" type="fixed">
       <parent link="${prefix}_HandPalmLink"/>
@@ -167,12 +149,5 @@
       <origin xyz="0.0 0.0445 0.0255" rpy="${-PI/2} 0 0" />
     </joint>
-    <link name="${prefix}_HandPalmMarkerBLink" >
-      <visual>
-        <origin xyz="0 0 0" rpy="0 0 0" />
-        <geometry>
-          <sphere radius="0.01"/>
-        </geometry>
-      </visual>
-    </link>
+    <link name="${prefix}_HandPalmMarkerBLink" />
     <joint name="${prefix}_HandPalmMarkerDJoint" type="fixed">
       <parent link="${prefix}_HandPalmLink"/>
@@ -180,12 +155,5 @@
       <origin xyz="0.0 -0.0445 0.0255" rpy="${PI/2} 0 0" />
     </joint>
-    <link name="${prefix}_HandPalmMarkerDLink" >
-      <visual>
-        <origin xyz="0 0 0" rpy="0 0 0" />
-        <geometry>
-          <sphere radius="0.01"/>
-        </geometry>
-      </visual>
-    </link>
+    <link name="${prefix}_HandPalmMarkerDLink" />
     <joint name="${prefix}_HandPalmJoint" type="fixed">
       <parent link="${parent}"/>
@@ -233,7 +201,22 @@
       <xacro:if value="$(arg collision_model_simplified)">
         <collision>
-          <origin xyz="0.03 0 0.005" rpy="0 0 0" />
-          <geometry>
-            <box size="${0.08+collision_model_enlargement*2} ${0.025+collision_model_enlargement*2} ${0.05+collision_model_enlargement*2}"/>
+          <origin xyz="0.0270798802376 0 0.00195854902267" rpy="0 0 0"/>
+          <geometry>
+            <box size="0.0752255320549 0.0278776362538 0.0362581014633"/>
+          </geometry>
+        </collision>
+        <collision>
+          <origin xyz="0.0493242815137 0 0.0150546580553" rpy="0 0 0"/>
+          <geometry>
+            <sphere radius="0.0196040868759"/>
+          </geometry>
+        </collision>
+      </xacro:if>
+      <!-- collision mesh used for grasp planning -->
+      <xacro:if value="$(arg collision_model_full)">
+        <collision>
+          <origin xyz="0 0 -0.0045" rpy="${0.5 * PI} 0 -${0.5 * PI}" />
+          <geometry>
+            <mesh filename="${homeDirectory}/meshes/firstFingerLink.stl"/>
           </geometry>
             <surface>
@@ -247,10 +230,58 @@
         </collision>
       </xacro:if>
+      </xacro:unless>
+    </link>
+    <gazebo reference="${prefix}_HandFinger${number}KnuckleOneLink">
+      <turnGravityOff>false</turnGravityOff>
+      <selfCollide>true</selfCollide>
+    </gazebo>
+    <joint name="${prefix}_HandFinger${number}KnuckleOneJoint" type="revolute">
+      <parent link="${prefix}_HandPalmLink"/>
+      <child link="${prefix}_HandFinger${number}KnuckleOneLink"/>
+      <origin xyz="${xyz}" rpy="${rpy}"/>
+      <axis xyz="${axis}"/>
+      <limit effort="2" lower="0" upper="${PI}" velocity="3.27"/>
+      <dynamics damping="0.1"/>
+    </joint>
+    <gazebo reference="${prefix}_HandFinger${number}KnuckleOneJoint">
+      <provideFeedback>true</provideFeedback>
+    </gazebo>
+  </xacro:macro>
+  <xacro:macro name="KnuckleTwo" params="parent prefix number xyz rpy">
+    <link name="${prefix}_HandFinger${number}KnuckleTwoLink">
+      <visual>
+        <origin xyz="0 0 0" rpy="${PI} ${0.5 * PI} 0" />
+        <geometry>
+          <mesh filename="${homeDirectory}/meshes/secondFingerLink.stl"/>
+        </geometry>
+        <material name="bh_HandGrey"/>
+      </visual>
+      <inertial>
+        <origin xyz="0.031720 0.001070 -0.000586" />
+        <mass value="0.057957" />
+        <inertia  ixx="0.00000461" ixy="0.00000003"  ixz="0.00000164"
+                                   iyy="0.00003590"  iyz="0.00000004"
+                                                     izz="0.00003682" />
+      </inertial>
+      <xacro:unless value="$(arg collision_model_no_hands)">
+      <!-- collision mesh used for whole arm motion planning -->
+      <xacro:if value="$(arg collision_model_simplified)">
+        <collision>
+          <origin xyz="0.0455318503082 0 0" rpy="0 0 0.0424077153578"/>
+          <geometry>
+            <box size="0.0572708845139 0.0259905532002 0.0224001407623"/>
+          </geometry>
+        </collision>
+      </xacro:if>
       <!-- collision mesh used for grasp planning -->
       <xacro:if value="$(arg collision_model_full)">
         <collision>
-          <origin xyz="0 0 -0.0045" rpy="${0.5 * PI} 0 -${0.5 * PI}" />
-          <geometry>
-            <mesh filename="${homeDirectory}/meshes/firstFingerLink.stl"/>
+<!--          <origin xyz="0 0 0" rpy="${PI} ${0.5 * PI} 0" />
+          <geometry>
+            <mesh filename="${homeDirectory}/meshes/secondFingerLink.stl"/>
+          </geometry>-->
+          <origin xyz="0.03 0 0" rpy="0 0 0" />
+          <geometry>
+            <box size="0.07 0.02 0.02" />
           </geometry>
             <surface>
@@ -265,77 +296,4 @@
       </xacro:if>
       </xacro:unless>
-    </link>
-    <gazebo reference="${prefix}_HandFinger${number}KnuckleOneLink">
-      <turnGravityOff>false</turnGravityOff>
-      <selfCollide>true</selfCollide>
-    </gazebo>
-    <joint name="${prefix}_HandFinger${number}KnuckleOneJoint" type="revolute">
-      <parent link="${prefix}_HandPalmLink"/>
-      <child link="${prefix}_HandFinger${number}KnuckleOneLink"/>
-      <origin xyz="${xyz}" rpy="${rpy}"/>
-      <axis xyz="${axis}"/>
-      <limit effort="2" lower="0" upper="${PI}" velocity="3.27"/>
-      <dynamics damping="0.1"/>
-    </joint>
-    <gazebo reference="${prefix}_HandFinger${number}KnuckleOneJoint">
-      <provideFeedback>true</provideFeedback>
-    </gazebo>
-  </xacro:macro>
-  <xacro:macro name="KnuckleTwo" params="parent prefix number xyz rpy">
-    <link name="${prefix}_HandFinger${number}KnuckleTwoLink">
-      <visual>
-        <origin xyz="0 0 0" rpy="${PI} ${0.5 * PI} 0" />
-        <geometry>
-          <mesh filename="${homeDirectory}/meshes/secondFingerLink.stl"/>
-        </geometry>
-        <material name="bh_HandGrey"/>
-      </visual>
-      <inertial>
-        <origin xyz="0.031720 0.001070 -0.000586" />
-        <mass value="0.057957" />
-        <inertia  ixx="0.00000461" ixy="0.00000003"  ixz="0.00000164"
-                                   iyy="0.00003590"  iyz="0.00000004"
-                                                     izz="0.00003682" />
-      </inertial>
-      <xacro:unless value="$(arg collision_model_no_hands)">
-      <!-- collision mesh used for whole arm motion planning -->
-      <xacro:if value="$(arg collision_model_simplified)">
-        <collision>
-          <origin xyz="0.03 0 0" rpy="0 0 0" />
-          <geometry>
-            <box size="${0.07+collision_model_enlargement*2} ${0.03+collision_model_enlargement*2} ${0.022+collision_model_enlargement*2}"/>
-          </geometry>
-            <surface>
-              <friction>
-                <ode>
-                  <mu>1.0</mu>
-                  <mu2>1.0</mu2>
-                </ode>
-              </friction>
-            </surface>
-        </collision>
-      </xacro:if>
-      <!-- collision mesh used for grasp planning -->
-      <xacro:if value="$(arg collision_model_full)">
-        <collision>
-<!--          <origin xyz="0 0 0" rpy="${PI} ${0.5 * PI} 0" />
-          <geometry>
-            <mesh filename="${homeDirectory}/meshes/secondFingerLink.stl"/>
-          </geometry>-->
-          <origin xyz="0.03 0 0" rpy="0 0 0" />
-          <geometry>
-            <box size="0.07 0.02 0.02" />
-          </geometry>
-            <surface>
-              <friction>
-                <ode>
-                  <mu>1.0</mu>
-                  <mu2>1.0</mu2>
-                </ode>
-              </friction>
-            </surface>
-        </collision>
-      </xacro:if>
-      </xacro:unless>
       <self_collision_checking>
         <origin xyz="0.03 0.0 0.0" rpy="0 1.57075 0"/>
@@ -403,16 +361,14 @@
       <xacro:if value="$(arg collision_model_simplified)">
         <collision>
-          <origin xyz="0.025 0 0" rpy="0 0 0" />
-          <geometry>
-            <box size="${0.07+collision_model_enlargement*2} ${0.02+collision_model_enlargement*2} ${0.022+collision_model_enlargement*2}"/>
-          </geometry>
-            <surface>
-              <friction>
-                <ode>
-                  <mu>1.0</mu>
-                  <mu2>1.0</mu2>
-                </ode>
-              </friction>
-            </surface>
+          <origin xyz="0.0220463573933 0 0" rpy="0 0 0"/>
+          <geometry>
+            <box size="0.0456312298775 0.0218328088522 0.0227420330048"/>
+          </geometry>
+        </collision>
+        <collision>
+          <origin xyz="0.046044960618 0.001 0" rpy="0 0 0"/>
+          <geometry>
+            <sphere radius="0.012090086937"/>
+          </geometry>
         </collision>
       </xacro:if>

Commit message: added 0 mass param for dummy links

File: barrett_hand_defs/defs/barret_hand.urdf.xacro (robot description, xacro)
@@ -137,5 +137,11 @@
       <origin xyz="0.0445 0.0 0.0255" rpy="0 ${PI/2} 0" />
     </joint>
-    <link name="${prefix}_HandPalmMarkerALink" />
+    <link name="${prefix}_HandPalmMarkerALink">
+      <inertial>
+        <mass value="0"/>
+        <origin rpy="0 0 0" xyz="0 0 0"/>
+        <inertia ixx="0" ixy="0" ixz="0" iyy="0" iyz="0" izz="0"/>
+      </inertial>
+    </link>
     <joint name="${prefix}_HandPalmMarkerCJoint" type="fixed">
       <parent link="${prefix}_HandPalmLink"/>
@@ -143,5 +149,11 @@
       <origin xyz="-0.0445 0.0 0.0255" rpy="0 ${-PI/2} 0" />
     </joint>
-    <link name="${prefix}_HandPalmMarkerCLink" />
+    <link name="${prefix}_HandPalmMarkerCLink">
+      <inertial>
+        <mass value="0"/>
+        <origin rpy="0 0 0" xyz="0 0 0"/>
+        <inertia ixx="0" ixy="0" ixz="0" iyy="0" iyz="0" izz="0"/>
+      </inertial>
+    </link>
     <joint name="${prefix}_HandPalmMarkerBJoint" type="fixed">
       <parent link="${prefix}_HandPalmLink"/>
@@ -149,5 +161,11 @@
       <origin xyz="0.0 0.0445 0.0255" rpy="${-PI/2} 0 0" />
     </joint>
-    <link name="${prefix}_HandPalmMarkerBLink" />
+    <link name="${prefix}_HandPalmMarkerBLink">
+      <inertial>
+        <mass value="0"/>
+        <origin rpy="0 0 0" xyz="0 0 0"/>
+        <inertia ixx="0" ixy="0" ixz="0" iyy="0" iyz="0" izz="0"/>
+      </inertial>
+    </link>
     <joint name="${prefix}_HandPalmMarkerDJoint" type="fixed">
       <parent link="${prefix}_HandPalmLink"/>
@@ -155,5 +173,11 @@
       <origin xyz="0.0 -0.0445 0.0255" rpy="${PI/2} 0 0" />
     </joint>
-    <link name="${prefix}_HandPalmMarkerDLink" />
+    <link name="${prefix}_HandPalmMarkerDLink">
+      <inertial>
+        <mass value="0"/>
+        <origin rpy="0 0 0" xyz="0 0 0"/>
+        <inertia ixx="0" ixy="0" ixz="0" iyy="0" iyz="0" izz="0"/>
+      </inertial>
+    </link>
     <joint name="${prefix}_HandPalmJoint" type="fixed">
       <parent link="${parent}"/>

Commit message: compatibility with new version of xacro

File: barrett_hand_defs/defs/barret_hand.urdf.xacro (robot description, xacro)
@@ -37,5 +37,5 @@
   <xacro:property name="highResModelDirectory" value="${homeDirectory}/meshes/splitModels" />
   <xacro:property name="PI" value="3.1415926535897931" />
-  <property name="collision_model_enlargement" value="$(arg collision_model_enlargement)" />
+  <xacro:property name="collision_model_enlargement" value="$(arg collision_model_enlargement)" />
   <xacro:macro name="palm" params="prefix parent *origin">
     <link name="${prefix}_HandPalmLink" >
@@ -183,5 +183,5 @@
       <parent link="${parent}"/>
       <child link="${prefix}_HandPalmLink"/>
-      <insert_block name="origin"/>
+      <xacro:insert_block name="origin"/>
       <provideFeedback value="true"/>
     </joint>
@@ -504,5 +504,5 @@
   <xacro:macro name="barret_hand" params="prefix parent *origin with_optoforce">
     <xacro:palm prefix="${prefix}" parent="${parent}">
-      <insert_block name="origin"/>
+      <xacro:insert_block name="origin"/>
     </xacro:palm>
     <xacro:fingers prefix="${prefix}" parent="${prefix}_HandPalmLink" number="Three" xyz="0 -0.05 0.0754" rpy="-${0.5 * PI} 0 -${0.5 * PI}" with_optoforce="${with_optoforce}"/>

File: barrett_hand_defs/defs/barret_hand_export.urdf.xacro (robot description, xacro)
@@ -82,5 +82,5 @@
             <parent link="${parent}"/>
             <child link="${prefix}_HandPalmLink"/>
-            <insert_block name="origin"/>
+            <xacro:insert_block name="origin"/>
             <provideFeedback value="true"/>
         </joint>
@@ -209,5 +209,5 @@
     <xacro:macro name="barret_hand" params="prefix parent *origin">
         <xacro:palm prefix="${prefix}" parent="${parent}">
-            <insert_block name="origin"/>
+            <xacro:insert_block name="origin"/>
         </xacro:palm>
         <xacro:fingers prefix="${prefix}" parent="${prefix}_HandPalmLink" number="Three" xyz="0 -0.05 0.0754" rpy="-${0.5 * PI} 0 -${0.5 * PI}"/>

Commit message: more natural colors for barretthand

File: barrett_hand_defs/defs/barret_hand.urdf.xacro (robot description, xacro)
@@ -29,5 +29,5 @@
        xmlns:interface="http://playerstage.sourceforge.net/gazebo/xmlschema/#interface"
        xmlns:xacro="http://www.ros.org/wiki/xacro">
-  <xacro:include filename="$(find barrett_hand_defs)/defs/materials.xml"/>
+  <!--<xacro:include filename="$(find barrett_hand_defs)/defs/materials.xml"/>-->
   <xacro:arg name="collision_model_full" default="true"/>
   <xacro:arg name="collision_model_simplified" default="false"/>
@@ -52,5 +52,7 @@
           <mesh filename="${homeDirectory}/meshes/palm.stl"/>
         </geometry>
-        <material name="bh_HandGrey"/>
+        <material name="Blue" >
+          <color rgba="0.2 0.2 0.9 1.0"/>
+        </material>
       </visual>
       <xacro:unless value="$(arg collision_model_no_hands)">
@@ -131,4 +133,5 @@
       <turnGravityOff>false</turnGravityOff>
       <selfCollide>true</selfCollide>
+      <material>Gazebo/Blue</material>
     </gazebo>
     <joint name="${prefix}_HandPalmMarkerAJoint" type="fixed">
@@ -212,5 +215,7 @@
           <mesh filename="${homeDirectory}/meshes/firstFingerLink.stl"/>
         </geometry>
-        <material name="bh_HandGrey"/>
+        <material name="LightBlue" >
+          <color rgba="0.5 0.5 1.0 1.0"/>
+        </material>
       </visual>
       <inertial>
@@ -259,4 +264,5 @@
       <turnGravityOff>false</turnGravityOff>
       <selfCollide>true</selfCollide>
+      <material>Gazebo/Grey</material>
     </gazebo>
     <joint name="${prefix}_HandFinger${number}KnuckleOneJoint" type="revolute">
@@ -279,5 +285,7 @@
           <mesh filename="${homeDirectory}/meshes/secondFingerLink.stl"/>
         </geometry>
-        <material name="bh_HandGrey"/>
+        <material name="LightBlue" >
+          <color rgba="0.5 0.5 1.0 1.0"/>
+        </material>
       </visual>
       <inertial>
@@ -338,4 +346,5 @@
       <turnGravityOff>false</turnGravityOff>
       <selfCollide>true</selfCollide>
+      <material>Gazebo/Grey</material>
     </gazebo>
     <joint name="${prefix}_HandFinger${number}KnuckleTwoJoint" type="revolute">
@@ -364,5 +373,7 @@
           </xacro:unless>
         </geometry>
-        <material name="bh_HandGrey"/>
+        <material name="LightBlue" >
+          <color rgba="0.5 0.5 1.0 1.0"/>
+        </material>
       </visual>
 <!--      <inertial>
@@ -435,4 +446,5 @@
       <turnGravityOff>false</turnGravityOff>
       <selfCollide>true</selfCollide>
+      <material>Gazebo/Grey</material>
     </gazebo>
     <joint name="${prefix}_HandFinger${number}KnuckleThreeJoint" type="revolute">

Commit message: better colors

File: barrett_hand_defs/defs/barret_hand.urdf.xacro (robot description, xacro)
@@ -53,5 +53,5 @@
         </geometry>
         <material name="Blue" >
-          <color rgba="0.2 0.2 0.9 1.0"/>
+          <color rgba="0 0.7 1 1.0"/>
         </material>
       </visual>
@@ -215,6 +215,6 @@
           <mesh filename="${homeDirectory}/meshes/firstFingerLink.stl"/>
         </geometry>
-        <material name="LightBlue" >
-          <color rgba="0.5 0.5 1.0 1.0"/>
+        <material name="Grey" >
+          <color rgba="0.8 0.8 0.8 1.0"/>
         </material>
       </visual>
@@ -285,6 +285,6 @@
           <mesh filename="${homeDirectory}/meshes/secondFingerLink.stl"/>
         </geometry>
-        <material name="LightBlue" >
-          <color rgba="0.5 0.5 1.0 1.0"/>
+        <material name="Grey" >
+          <color rgba="0.8 0.8 0.8 1.0"/>
         </material>
       </visual>
@@ -373,6 +373,6 @@
           </xacro:unless>
         </geometry>
-        <material name="LightBlue" >
-          <color rgba="0.5 0.5 1.0 1.0"/>
+        <material name="Grey" >
+          <color rgba="0.8 0.8 0.8 1.0"/>
         </material>
       </visual>
